Commit message: remove unnecessary fixed joints

File: assets/yam.urdf (robot description, URDF)
Before this commit: robot converted_robot, 22 links, 21 joints
Links:
- removed link joint1_jointbody
- removed link joint2_jointbody
- removed link joint3_jointbody
- removed link joint4_jointbody
- removed link joint5_jointbody
- removed link joint6_jointbody
- removed link left_finger_jointbody
- removed link right_finger_jointbody
- removed link world
Joints:
- removed joint joint1_offset
- removed joint joint2_offset
- removed joint joint3_offset
- removed joint joint4_offset
- removed joint joint5_offset
- removed joint joint6_offset
- removed joint left_finger_offset
- removed joint right_finger_offset
- removed joint world2arm_fixed
- joint joint1: child joint1_jointbody -> link_1
- joint joint2: child joint2_jointbody -> link_2
- joint joint3: child joint3_jointbody -> link_3
- joint joint4: child joint4_jointbody -> link_4
- joint joint5: child joint5_jointbody -> link_5
- joint joint6: child joint6_jointbody -> link_6
- joint left_finger: child left_finger_jointbody -> link_left_finger
- joint right_finger: child right_finger_jointbody -> link_right_finger

Commit message: better collision models

File: assets/yam.urdf (robot description, URDF)
Before this commit: robot i2rt_yam, 13 links, 12 joints
Links:
- removed link lf_down
- removed link lf_rot
- removed link rf_down
- removed link rf_rot
- link arm: geometry collision cylinder length=0.097728589 radius=0.033; visual mesh filename=meshes/converted_model2_404040ff.obj
- link link_1: geometry collision mesh filename=meshes/converted_model2__2_404040ff.obj; visual mesh filename=meshes/converted_model2__2_404040ff.obj
- link link_2: geometry collision mesh filename=meshes/converted_model2__3_404040ff.obj; collision mesh filename=meshes/converted_model2__4_404040ff.obj
- link link_3: geometry collision mesh filename=meshes/converted_model2__6_404040ff.obj; collision mesh filename=meshes/converted_model2__7_404040ff.obj
- link link_4: geometry collision cylinder length=0.05 radius=0.03; visual mesh filename=meshes/converted_model2__10_404040ff.obj
- link link_5: geometry collision cylinder length=0.05 radius=0.03; visual mesh filename=meshes/converted_model2__11_404040ff.obj
- link link_6: geometry collision cylinder length=0.055 radius=0.03; visual mesh filename=meshes/converted_model2__12_404040ff.obj
- link link_left_finger: geometry collision mesh filename=meshes/converted_model2__14_404040ff.obj; collision mesh filename=meshes/converted_model2__15_404040ff.obj
- link link_right_finger: geometry collision mesh filename=meshes/converted_model2__16_404040ff.obj; collision mesh filename=meshes/converted_model2__17_404040ff.obj
Joints:
- removed joint lf_rot2lf_down_fixed
- removed joint link_left_finger2lf_rot_fixed
- removed joint link_right_finger2rf_rot_fixed
- removed joint rf_rot2rf_down_fixed
- joint joint1: origin xyz=0.0 0.0 0.0631 rpy=0.0 0.0 1.5707963267948963 -> xyz=0.0 0.0 0.074642863 rpy=0.0 0.0 1.5707963267948963

Commit message: better file names

File: assets/yam.urdf (robot description, URDF)
Before this commit: robot i2rt_yam, 9 links, 8 joints
Links:
- link arm: geometry collision cylinder length=0.097728589 radius=0.033; visual mesh filename=meshes/arm.obj
- link link_1: geometry collision mesh filename=meshes/link_1.obj; visual mesh filename=meshes/link_1.obj
- link link_2: geometry collision mesh filename=meshes/link_2_1.obj; collision mesh filename=meshes/link_2_2.obj
- link link_3: geometry collision mesh filename=meshes/link_3_1.obj; collision mesh filename=meshes/link_3_2.obj
- link link_4: geometry collision cylinder length=0.05 radius=0.03; visual mesh filename=meshes/link_4.obj
- link link_5: geometry collision cylinder length=0.05 radius=0.03; visual mesh filename=meshes/link_5.obj
- link link_6: geometry collision cylinder length=0.055 radius=0.03; visual mesh filename=meshes/link_6_1.obj
- link link_left_finger: geometry collision mesh filename=meshes/link_left_finger_1.obj; collision mesh filename=meshes/link_left_finger_2.obj
- link link_right_finger: geometry collision mesh filename=meshes/link_right_finger_1.obj; collision mesh filename=meshes/link_right_finger_2.obj
